File: Schematic/Fob.sch (KiCad schematic (older format))
At the start: 14 parts, among them IC1 ATMEGA328-P, P1 RF24L01, P2 ICSP, SW1 SW_PUSH, SW2 SW_PUSH

Commit message: PCB: version 2
Parts:
- removed D1: Led_Small, LEDs:LED-3MM, symbol Led_Small
- removed R3: 330, Resistors_ThroughHole:Resistor_Horizontal_RM7mm, symbol R
- removed SW2: SW_PUSH, fob:SW_PUSH_6mm, symbol SW_PUSH
- C1, C2, C3: footprint fob:C_Disc_P5 -> fob:C_Disc_P2
- C4: footprint Capacitors_ThroughHole:C_Radial_D5_L6_P2.5 -> fob:C_Radial_D5_L6_P2.5_length
- IC1: footprint Housings_QFP:TQFP-32_7x7mm_Pitch0.8mm -> fob:TQFP-32_7x7mm_Pitch0.8mm
Connections:
- net at R2.2, SW1.1: now also IC1.9 ((PCINT21/OC0B/T1)PD5); no longer IC1.32 ((PCINT18/INT0)PD2)
Changed lines of the file:
@@
 F 0 "IC1" H 5000 4500 50  0000 L BNN
 F 1 "ATMEGA328-P" H 6150 1850 50  0000 L BNN
-F 2 "Housings_QFP:TQFP-32_7x7mm_Pitch0.8mm" H 5750 3250 50  0000 C CIN
+F 2 "fob:TQFP-32_7x7mm_Pitch0.8mm" H 5750 3250 50  0000 C CIN
 F 3 "" H 5750 3250 50  0000 C CNN
 	1    5750 3250
@@
 $EndComp
 $Comp
-L Led_Small D1
-U 1 1 56D1ACC8
-P 7700 3750
-F 0 "D1" H 7650 3875 50  0000 L CNN
-F 1 "Led_Small" H 7525 3650 50  0000 L CNN
-F 2 "LEDs:LED-3MM" V 7700 3750 50  0001 C CNN
-F 3 "" V 7700 3750 50  0000 C CNN
-	1    7700 3750
-	-1   0    0    1
-$EndComp
-$Comp
 L R R2
 U 1 1 56D1AD6E
@@
 	1    7450 3950
 	0    1    1    0
-$EndComp
-$Comp
-L R R3
-U 1 1 56D1ADE5
-P 7300 3750
-F 0 "R3" V 7380 3750 50  0000 C CNN
-F 1 "330" V 7300 3750 50  0000 C CNN
-F 2 "Resistors_ThroughHole:Resistor_Horizontal_RM7mm" V 7230 3750 50  0001 C CNN
-F 3 "" H 7300 3750 50  0000 C CNN
-	1    7300 3750
-	0    -1   -1   0
 $EndComp
 $Comp
@@
 F 0 "C1" H 4610 2370 50  0000 L CNN
 F 1 "100n" H 4610 2220 50  0000 L CNN
-F 2 "fob:C_Disc_P5" H 4600 2300 50  0001 C CNN
+F 2 "fob:C_Disc_P2" H 4600 2300 50  0001 C CNN
 F 3 "" H 4600 2300 50  0000 C CNN
 	1    4600 2300
@@
 F 0 "C2" H 4760 2670 50  0000 L CNN
 F 1 "100n" H 4760 2520 50  0000 L CNN
-F 2 "fob:C_Disc_P5" H 4750 2600 50  0001 C CNN
+F 2 "fob:C_Disc_P2" H 4750 2600 50  0001 C CNN
 F 3 "" H 4750 2600 50  0000 C CNN
 	1    4750 2600
@@
 NoConn ~ 6750 4050
 NoConn ~ 6750 4150
-NoConn ~ 6750 4250
 NoConn ~ 6750 4350
 NoConn ~ 6750 4450
@@
 F 0 "C3" H 4660 3020 50  0000 L CNN
 F 1 "100n" H 4660 2870 50  0000 L CNN
-F 2 "fob:C_Disc_P5" H 4650 2950 50  0001 C CNN
+F 2 "fob:C_Disc_P2" H 4650 2950 50  0001 C CNN
 F 3 "" H 4650 2950 50  0000 C CNN
 	1    4650 2950
@@
 	7200 3600 7400 3600
 Wire Wire Line
-	6750 3950 7300 3950
+	7000 3950 7300 3950
 Wire Wire Line
 	7600 3950 8000 3950
 Wire Wire Line
 	7200 4200 7200 3950
-Connection ~ 7200 3950
 Wire Wire Line
 	7200 4800 7200 4950
@@
 	8650 1650 8650 2450
 Wire Wire Line
-	9300 2650 9300 3350
-Wire Wire Line
-	9300 3350 6850 3350
+	9300 3350 9300 2650
+Wire Wire Line
+	6850 3350 9300 3350
 Wire Wire Line
 	6850 3350 6850 3600
@@
 Wire Wire Line
 	9300 2150 9300 2000
-Wire Wire Line
-	7800 3750 8000 3750
-Wire Wire Line
-	8000 3750 8000 3950
-Wire Wire Line
-	7450 3750 7600 3750
-Wire Wire Line
-	6750 3750 7150 3750
 NoConn ~ 6750 2150
 NoConn ~ 5000 2000
-NoConn ~ 6950 4000
 NoConn ~ 6700 2250
 NoConn ~ 6900 2150
@@
 F 0 "C4" H 2010 2770 50  0000 L CNN
 F 1 "10uF" H 2010 2620 50  0000 L CNN
-F 2 "Capacitors_ThroughHole:C_Radial_D5_L6_P2.5" H 2000 2700 50  0001 C CNN
+F 2 "fob:C_Radial_D5_L6_P2.5_length" H 2000 2700 50  0001 C CNN
 F 3 "" H 2000 2700 50  0000 C CNN
 	1    2000 2700
@@
 	2000 3000 2400 3000
 Connection ~ 2400 3000
-$Comp
-L SW_PUSH SW2
-U 1 1 56DAD8F4
-P 8700 4350
-F 0 "SW2" H 8850 4460 50  0000 C CNN
-F 1 "SW_PUSH" H 8700 4270 50  0000 C CNN
-F 2 "fob:SW_PUSH_6mm" H 8700 4350 50  0001 C CNN
-F 3 "" H 8700 4350 50  0000 C CNN
-	1    8700 4350
-	0    1    1    0
-$EndComp
-$Comp
-L GND #PWR017
-U 1 1 56DAD958
-P 8700 4850
-F 0 "#PWR017" H 8700 4600 50  0001 C CNN
-F 1 "GND" H 8700 4700 50  0000 C CNN
-F 2 "" H 8700 4850 50  0000 C CNN
-F 3 "" H 8700 4850 50  0000 C CNN
-	1    8700 4850
-	1    0    0    -1
-$EndComp
-Wire Wire Line
-	8700 4850 8700 4650
-Wire Wire Line
-	8700 3350 8700 4050
-Connection ~ 8700 3350
+NoConn ~ 6750 3750
+NoConn ~ 6750 3950
+Wire Wire Line
+	6750 4250 7000 4250
+Wire Wire Line
+	7000 4250 7000 3950
+Connection ~ 7200 3950
 $EndSCHEMATC
